File: JustType.kicad_sch (KiCad schematic)
At the start: 56 parts, among them J1 Conn_01x02, J2 Conn_01x02, SW1 SW_Push, SW10 SW_Push, SW11 SW_Push, SW12 SW_Push, SW13 SW_Push, SW14 SW_Push, SW15 SW_Push, SW16 SW_Push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

Commit message: v4
Parts:
- removed D10, D15, D20, D25, D4, D5, D9: 1N4448W, Diode_SMD:D_SOD-123, symbol Diode:1N4448W
- removed J1, J2: Conn_01x02, Connector_JST:JST_PH_S2B-PH-K_1x02_P2.00mm_Horizontal, symbol Connector_Generic:Conn_01x02
- removed RV1, RV2: R_Potentiometer_Dual, keyboard_jsa:PSP thumbstick, symbol Device:R_Potentiometer_Dual
- removed SW10, SW15, SW19'1, SW20, SW25, SW4, SW5, SW9: SW_Push, keyboard_jsa:ChocV1_Hotswap, symbol Switch:SW_Push
- added D12, D18, D22, D6: 1N4448W, keyboard_jsa:D3_SMD_v2, symbol Diode:1N4448W
- added SW12, SW18, SW22, SW6: SW_Push, keyboard_jsa:ChocV1_Solder, symbol Switch:SW_Push
- D1: footprint Diode_SMD:D_SOD-123 -> keyboard_jsa:D3_SMD_v2
- D10: renamed from D17; footprint Diode_SMD:D_SOD-123 -> keyboard_jsa:D3_SMD_v2
- D11: renamed from D22; footprint Diode_SMD:D_SOD-123 -> keyboard_jsa:D3_SMD_v2
- D13: renamed from D3; footprint Diode_SMD:D_SOD-123 -> keyboard_jsa:D3_SMD_v2
- D14: renamed from D8; footprint Diode_SMD:D_SOD-123 -> keyboard_jsa:D3_SMD_v2
- D15: renamed from D13; footprint Diode_SMD:D_SOD-123 -> keyboard_jsa:D3_SMD_v2
- D16: renamed from D18; footprint Diode_SMD:D_SOD-123 -> keyboard_jsa:D3_SMD_v2
- D17: renamed from D23; footprint Diode_SMD:D_SOD-123 -> keyboard_jsa:D3_SMD_v2
- D19: renamed from D14; footprint Diode_SMD:D_SOD-123 -> keyboard_jsa:D3_SMD_v2
- D2: renamed from D6; footprint Diode_SMD:D_SOD-123 -> keyboard_jsa:D3_SMD_v2
- D20: renamed from D19; footprint Diode_SMD:D_SOD-123 -> keyboard_jsa:D3_SMD_v2
- D21: renamed from D24; footprint Diode_SMD:D_SOD-123 -> keyboard_jsa:D3_SMD_v2
- D3: renamed from D11; footprint Diode_SMD:D_SOD-123 -> keyboard_jsa:D3_SMD_v2
- D4: renamed from D16; footprint Diode_SMD:D_SOD-123 -> keyboard_jsa:D3_SMD_v2
- D5: renamed from D21; footprint Diode_SMD:D_SOD-123 -> keyboard_jsa:D3_SMD_v2
- D7: renamed from D2; footprint Diode_SMD:D_SOD-123 -> keyboard_jsa:D3_SMD_v2
- D8: renamed from D7; footprint Diode_SMD:D_SOD-123 -> keyboard_jsa:D3_SMD_v2
- D9: renamed from D12; footprint Diode_SMD:D_SOD-123 -> keyboard_jsa:D3_SMD_v2
- SW1: footprint keyboard_jsa:ChocV1_Hotswap -> keyboard_jsa:ChocV1_Solder
- SW10: renamed from SW17; footprint keyboard_jsa:ChocV1_Hotswap -> keyboard_jsa:ChocV1_Solder
- SW11: renamed from SW22; footprint keyboard_jsa:ChocV1_Hotswap -> keyboard_jsa:ChocV1_Solder
- SW13: renamed from SW3; footprint keyboard_jsa:ChocV1_Hotswap -> keyboard_jsa:ChocV1_Solder
- SW14: renamed from SW8; footprint keyboard_jsa:ChocV1_Hotswap -> keyboard_jsa:ChocV1_Solder
- SW15: renamed from SW13; footprint keyboard_jsa:ChocV1_Hotswap -> keyboard_jsa:ChocV1_Solder
- SW16: renamed from SW18; footprint keyboard_jsa:ChocV1_Hotswap -> keyboard_jsa:ChocV1_Solder
- SW17: renamed from SW23; footprint keyboard_jsa:ChocV1_Hotswap -> keyboard_jsa:ChocV1_Solder
- SW19: renamed from SW14; footprint keyboard_jsa:ChocV1_Hotswap -> keyboard_jsa:ChocV1_Solder
- SW2: renamed from SW6; footprint keyboard_jsa:ChocV1_Hotswap -> keyboard_jsa:ChocV1_Solder
- SW20: renamed from SW19; footprint keyboard_jsa:ChocV1_Hotswap -> keyboard_jsa:ChocV1_Solder
- SW21: renamed from SW24; footprint keyboard_jsa:ChocV1_Hotswap -> keyboard_jsa:ChocV1_Solder
- SW3: renamed from SW11; footprint keyboard_jsa:ChocV1_Hotswap -> keyboard_jsa:ChocV1_Solder
- SW4: renamed from SW16; footprint keyboard_jsa:ChocV1_Hotswap -> keyboard_jsa:ChocV1_Solder
- SW5: renamed from SW21; footprint keyboard_jsa:ChocV1_Hotswap -> keyboard_jsa:ChocV1_Solder
- SW7: renamed from SW2; footprint keyboard_jsa:ChocV1_Hotswap -> keyboard_jsa:ChocV1_Solder
- SW8: renamed from SW7; footprint keyboard_jsa:ChocV1_Hotswap -> keyboard_jsa:ChocV1_Solder
- SW9: renamed from SW12; footprint keyboard_jsa:ChocV1_Hotswap -> keyboard_jsa:ChocV1_Solder
Connections:
- net Row 5 is gone; now on net Row 4: U1.9 (6/PD7)
- net Col 1: now also U1.2 (RX1/PD2), SW12.1, SW18.1, SW22.1, SW6.1; no longer SW1.1, SW13.1, SW7.1, U1.12 (9/PB5)
- net Col 2: now also SW11.1, SW17.1, SW21.1, SW5.1, U1.6 (3/PD0); no longer SW14.1, SW2.1, SW8.1, U1.11 (8/PB4)
- net Col 3: now also SW10.1, SW16.1, SW20.1, SW4.1, U1.8 (5/PC6); no longer SW15.1, SW19.1, SW3.1, SW9.1, U1.10 (7/PE6)
- net Col 4: now also SW15.1, SW19.1, SW3.1, SW9.1, U1.10 (7/PE6); no longer SW10.1, SW16.1, SW20.1, SW4.1, U1.16 (15/PB1)
- net Col 5: now also SW14.1, SW2.1, SW8.1, U1.12 (9/PB5); no longer SW11.1, SW17.1, SW21.1, SW5.1, U1.15 (14/PB3)
- net Row 1: now also U1.1 (TX0/PD3), D6.2 (A); no longer U1.5 (2/PD1)
- net Row 2: now also U1.5 (2/PD1), D12.2 (A); no longer U1.6 (3/PD0)
- net Row 3: now also D18.2 (A)
- net Row 4: now also D22.2 (A); no longer U1.8 (5/PC6)
- net BAT+: no longer names the net of U1.24 (RAW)
- net X: no longer names the net of U1.17 (A0/PF7)
- net Y: no longer names the net of U1.18 (A1/PF6)
- new net: D18.1 (K), SW18.2
- new net: D12.1 (K), SW12.2
- new net: D22.1 (K), SW22.2
- new net: D6.1 (K), SW6.2
- new net Col 6: SW1.1, SW13.1, SW7.1, U1.11 (8/PB4)
- no-connect marks 7 -> 10
Other:
- moved on the sheet: SW20

Commit message: R5 validated.
Parts:
- added H1: MountingHole, MountingHole:MountingHole_3.2mm_M3, symbol Mechanical:MountingHole
- D1, D10, D11, D12, D13, D14, D15, D16, D17, D18, D19, D2, D20, D21, D22, D3, D4, D5, D6, D7, D8, D9: footprint keyboard_jsa:D3_SMD_v2 -> keyboard_jsa:D3_SMD_v2_Reverse
- SW1, SW10, SW11, SW12, SW13, SW14, SW15, SW16, SW17, SW18, SW19, SW2, SW20, SW21, SW22, SW3, SW4, SW5, SW6, SW7, SW8, SW9: footprint keyboard_jsa:ChocV1_Solder -> keyboard_jsa:ChocV1_Solder_Reverse
Changed lines of the file:
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@@
 			)
 		)
-		(property "Footprint" "keyboard_jsa:D3_SMD_v2"
+		(property "Footprint" "keyboard_jsa:D3_SMD_v2_Reverse"
 			(at 221.615 90.17 0)
 			(effects
@@
 			)
 		)
-		(property "Footprint" "keyboard_jsa:ChocV1_Solder"
+		(property "Footprint" "keyboard_jsa:ChocV1_Solder_Reverse"
 			(at 190.5 63.5 0)
 			(effects
@@
 			)
 		)
-		(property "Footprint" "keyboard_jsa:D3_SMD_v2"
+		(property "Footprint" "keyboard_jsa:D3_SMD_v2_Reverse"
 			(at 206.375 90.17 0)
 			(effects
@@
 			)
 		)
-		(property "Footprint" "keyboard_jsa:ChocV1_Solder"
+		(property "Footprint" "keyboard_jsa:ChocV1_Solder_Reverse"
 			(at 160.02 45.72 0)
 			(effects
@@
 	)
 	(symbol
+		(lib_id "Mechanical:MountingHole")
+		(at 179.07 153.67 0)
+		(unit 1)
+		(exclude_from_sim yes)
+		(in_bom no)
+		(on_board yes)
+		(dnp no)
+		(fields_autoplaced yes)
+		(property "Reference" "H1"
+			(at 181.61 152.3999 0)
+			(effects
+				(font
+					(size 1.27 1.27)
+				)
+				(justify left)
+			)
+		)
+		(property "Value" "MountingHole"
+			(at 181.61 154.9399 0)
+			(effects
+				(font
+					(size 1.27 1.27)
+				)
+				(justify left)
+			)
+		)
+		(property "Footprint" "MountingHole:MountingHole_3.2mm_M3"
+			(at 179.07 153.67 0)
+			(effects
+				(font
+					(size 1.27 1.27)
+				)
+				(hide yes)
+			)
+		)
+		(property "Datasheet" "~"
+			(at 179.07 153.67 0)
+			(effects
+				(font
+					(size 1.27 1.27)
+				)
+				(hide yes)
+			)
+		)
+		(property "Description" "Mounting Hole without connection"
+			(at 179.07 153.67 0)
+			(effects
+				(font
+					(size 1.27 1.27)
+				)
+				(hide yes)
+			)
+		)
+		(instances
+			(project ""
+				(path "/6e8e757a-c6cb-4b52-bdb0-ff823309d752"
+					(reference "H1")
+					(unit 1)
+				)
+			)
+		)
+	)
+	(symbol
 		(lib_id "Diode:1N4448W")
 		(at 165.1 54.61 270)
@@
 			)
 		)
-		(property "Footprint" "keyboard_jsa:D3_SMD_v2"
+		(property "Footprint" "keyboard_jsa:D3_SMD_v2_Reverse"
 			(at 160.655 54.61 0)
 			(effects
@@
 			)
 		)
-		(property "Footprint" "keyboard_jsa:D3_SMD_v2"
+		(property "Footprint" "keyboard_jsa:D3_SMD_v2_Reverse"
 			(at 221.615 72.39 0)
 			(effects
@@
 			)
 		)
-		(property "Footprint" "keyboard_jsa:D3_SMD_v2"
+		(property "Footprint" "keyboard_jsa:D3_SMD_v2_Reverse"
 			(at 145.415 54.61 0)
 			(effects
@@
 			)
 		)
-		(property "Footprint" "keyboard_jsa:D3_SMD_v2"
+		(property "Footprint" "keyboard_jsa:D3_SMD_v2_Reverse"
 			(at 191.135 54.61 0)
 			(effects
@@
 			)
 		)
-		(property "Footprint" "keyboard_jsa:D3_SMD_v2"
+		(property "Footprint" "keyboard_jsa:D3_SMD_v2_Reverse"
 			(at 191.135 107.95 0)
 			(effects
@@
 			)
 		)
-		(property "Footprint" "keyboard_jsa:ChocV1_Solder"
+		(property "Footprint" "keyboard_jsa:ChocV1_Solder_Reverse"
 			(at 175.26 63.5 0)
 			(effects
@@
 			)
 		)
-		(property "Footprint" "keyboard_jsa:ChocV1_Solder"
+		(property "Footprint" "keyboard_jsa:ChocV1_Solder_Reverse"
 			(at 205.74 63.5 0)
 			(effects
@@
 			)
 		)
-		(property "Footprint" "keyboard_jsa:ChocV1_Solder"
+		(property "Footprint" "keyboard_jsa:ChocV1_Solder_Reverse"
 			(at 220.98 81.28 0)
 			(effects
@@
 			)
 		)
-		(property "Footprint" "keyboard_jsa:ChocV1_Solder"
+		(property "Footprint" "keyboard_jsa:ChocV1_Solder_Reverse"
 			(at 190.5 81.28 0)
 			(effects
@@
 			)
 		)
-		(property "Footprint" "keyboard_jsa:ChocV1_Solder"
+		(property "Footprint" "keyboard_jsa:ChocV1_Solder_Reverse"
 			(at 160.02 81.28 0)
 			(effects
@@
 			)
 		)
-		(property "Footprint" "keyboard_jsa:ChocV1_Solder"
+		(property "Footprint" "keyboard_jsa:ChocV1_Solder_Reverse"
 			(at 205.74 45.72 0)
 			(effects
@@
 			)
 		)
-		(property "Footprint" "keyboard_jsa:D3_SMD_v2"
+		(property "Footprint" "keyboard_jsa:D3_SMD_v2_Reverse"
 			(at 206.375 107.95 0)
 			(effects
@@
 			)
 		)
-		(property "Footprint" "keyboard_jsa:D3_SMD_v2"
+		(property "Footprint" "keyboard_jsa:D3_SMD_v2_Reverse"
 			(at 160.655 72.39 0)
 			(effects
@@
 			)
 		)
-		(property "Footprint" "keyboard_jsa:ChocV1_Solder"
+		(property "Footprint" "keyboard_jsa:ChocV1_Solder_Reverse"
 			(at 190.5 99.06 0)
 			(effects
@@
 			)
 		)
-		(property "Footprint" "keyboard_jsa:ChocV1_Solder"
+		(property "Footprint" "keyboard_jsa:ChocV1_Solder_Reverse"
 			(at 160.02 63.5 0)
 			(effects
@@
 			)
 		)
-		(property "Footprint" "keyboard_jsa:D3_SMD_v2"
+		(property "Footprint" "keyboard_jsa:D3_SMD_v2_Reverse"
 			(at 175.895 90.17 0)
 			(effects
@@
 			)
 		)
-		(property "Footprint" "keyboard_jsa:D3_SMD_v2"
+		(property "Footprint" "keyboard_jsa:D3_SMD_v2_Reverse"
 			(at 206.375 72.39 0)
 			(effects
@@
 			)
 		)
-		(property "Footprint" "keyboard_jsa:D3_SMD_v2"
+		(property "Footprint" "keyboard_jsa:D3_SMD_v2_Reverse"
 			(at 175.895 107.95 0)
 			(effects
@@
 			)
 		)
-		(property "Footprint" "keyboard_jsa:D3_SMD_v2"
+		(property "Footprint" "keyboard_jsa:D3_SMD_v2_Reverse"
 			(at 145.415 90.17 0)
 			(effects
@@
 			)
 		)
-		(property "Footprint" "keyboard_jsa:ChocV1_Solder"
+		(property "Footprint" "keyboard_jsa:ChocV1_Solder_Reverse"
 			(at 144.78 45.72 0)
 			(effects
@@
 			)
 		)
-		(property "Footprint" "keyboard_jsa:ChocV1_Solder"
+		(property "Footprint" "keyboard_jsa:ChocV1_Solder_Reverse"
 			(at 175.26 99.06 0)
 			(effects
@@
 			)
 		)
-		(property "Footprint" "keyboard_jsa:D3_SMD_v2"
+		(property "Footprint" "keyboard_jsa:D3_SMD_v2_Reverse"
 			(at 206.375 54.61 0)
 			(effects
@@
 			)
 		)
-		(property "Footprint" "keyboard_jsa:ChocV1_Solder"
+		(property "Footprint" "keyboard_jsa:ChocV1_Solder_Reverse"
 			(at 220.98 99.06 0)
 			(effects
@@
 			)
 		)
-		(property "Footprint" "keyboard_jsa:ChocV1_Solder"
+		(property "Footprint" "keyboard_jsa:ChocV1_Solder_Reverse"
 			(at 175.26 45.72 0)
 			(effects
@@
 			)
 		)
-		(property "Footprint" "keyboard_jsa:D3_SMD_v2"
+		(property "Footprint" "keyboard_jsa:D3_SMD_v2_Reverse"
 			(at 221.615 107.95 0)
 			(effects
@@
 			)
 		)
-		(property "Footprint" "keyboard_jsa:ChocV1_Solder"
+		(property "Footprint" "keyboard_jsa:ChocV1_Solder_Reverse"
 			(at 205.74 99.06 0)
 			(effects
@@
 			)
 		)
-		(property "Footprint" "keyboard_jsa:D3_SMD_v2"
+		(property "Footprint" "keyboard_jsa:D3_SMD_v2_Reverse"
 			(at 191.135 90.17 0)
 			(effects
@@
 			)
 		)
-		(property "Footprint" "keyboard_jsa:ChocV1_Solder"
+		(property "Footprint" "keyboard_jsa:ChocV1_Solder_Reverse"
 			(at 144.78 81.28 0)
 			(effects
@@
 			)
 		)
-		(property "Footprint" "keyboard_jsa:D3_SMD_v2"
+		(property "Footprint" "keyboard_jsa:D3_SMD_v2_Reverse"
 			(at 221.615 54.61 0)
 			(effects
@@
 			)
 		)
-		(property "Footprint" "keyboard_jsa:D3_SMD_v2"
+		(property "Footprint" "keyboard_jsa:D3_SMD_v2_Reverse"
 			(at 191.135 72.39 0)
 			(effects
@@
 			)
 		)
-		(property "Footprint" "keyboard_jsa:D3_SMD_v2"
+		(property "Footprint" "keyboard_jsa:D3_SMD_v2_Reverse"
 			(at 175.895 72.39 0)
 			(effects
@@
 			)
 		)
-		(property "Footprint" "keyboard_jsa:D3_SMD_v2"
+		(property "Footprint" "keyboard_jsa:D3_SMD_v2_Reverse"
 			(at 160.655 90.17 0)
 			(effects
@@
 			)
 		)
-		(property "Footprint" "keyboard_jsa:D3_SMD_v2"
+		(property "Footprint" "keyboard_jsa:D3_SMD_v2_Reverse"
 			(at 175.895 54.61 0)
 			(effects
@@
 			)
 		)
-		(property "Footprint" "keyboard_jsa:ChocV1_Solder"
+		(property "Footprint" "keyboard_jsa:ChocV1_Solder_Reverse"
 			(at 220.98 45.72 0)
 			(effects
@@
 			)
 		)
-		(property "Footprint" "keyboard_jsa:ChocV1_Solder"
+		(property "Footprint" "keyboard_jsa:ChocV1_Solder_Reverse"
 			(at 220.98 63.5 0)
 			(effects
@@
 			)
 		)
-		(property "Footprint" "keyboard_jsa:ChocV1_Solder"
+		(property "Footprint" "keyboard_jsa:ChocV1_Solder_Reverse"
 			(at 190.5 45.72 0)
 			(effects
@@
 			)
 		)
-		(property "Footprint" "keyboard_jsa:ChocV1_Solder"
+		(property "Footprint" "keyboard_jsa:ChocV1_Solder_Reverse"
 			(at 205.74 81.28 0)
 			(effects
@@
 			)
 		)
-		(property "Footprint" "keyboard_jsa:ChocV1_Solder"
+		(property "Footprint" "keyboard_jsa:ChocV1_Solder_Reverse"
 			(at 175.26 81.28 0)
 			(effects
@@
 			)
 		)
-		(property "Footprint" "keyboard_jsa:ChocV1_Solder"
+		(property "Footprint" "keyboard_jsa:ChocV1_Solder_Reverse"
 			(at 144.78 63.5 0)
 			(effects
@@
 			)
 		)
-		(property "Footprint" "keyboard_jsa:D3_SMD_v2"
+		(property "Footprint" "keyboard_jsa:D3_SMD_v2_Reverse"
 			(at 145.415 72.39 0)
 			(effects

Commit message: validating
Parts:
- SW1, SW10, SW11, SW12, SW13, SW14, SW15, SW16, SW17, SW18, SW19, SW2, SW20, SW21, SW22, SW3, SW4, SW5, SW6, SW7, SW8, SW9: footprint keyboard_jsa:ChocV1_Solder_Reverse -> keyboard_jsa:ChocV2_Solder_2side_v1
Connections:
- removed net GND: U1.23 (GND), U1.3 (GND), U1.4 (GND)
- net VCC: no longer names the net of U1.21 (VCC)
- no-connect marks 10 -> 14
